Commit message: fix IK and do mini hops with pos control

File: ros2_ws/src/robot_description/description/position_control.xacro (robot description, xacro)
@@ -16,5 +16,5 @@
             <cmd_min>-100</cmd_min>
             <cmd_offset>0.0</cmd_offset>
-            <initial_position>-0.3</initial_position>
+            <!-- <initial_position>-0.3</initial_position> -->
         </plugin>
         <plugin
@@ -32,5 +32,5 @@
             <cmd_min>-100</cmd_min>
             <cmd_offset>0.0</cmd_offset>
-            <initial_position>0.6</initial_position>
+            <!-- <initial_position>0.6</initial_position> -->
         </plugin>
     </gazebo>

File: ros2_ws/src/robot_description/description/robot.urdf.xacro (robot description, xacro)
@@ -84,4 +84,5 @@
     <!-- This has to be a revolute joint for some dumb reason -->
     <!-- Can also change this manually in the sdf to a fixed joint -->
+    <!-- <joint name="contact_joint" type="fixed"> -->
     <joint name="contact_joint" type="revolute">
         <parent link="knee_link" />
@@ -90,4 +91,5 @@
         <axis xyz="0 0 1" />
         <limit effort="1e-5" lower="0" upper="0" velocity="1e-5" />
+        <dynamics damping="0.1" friction="0.1" />
     </joint>
     <link name="foot_link">

Commit message: fix contact sensor not working, update jacobian

File: ros2_ws/src/robot_description/description/position_control.xacro (robot description, xacro)
@@ -8,13 +8,12 @@
             <use_force_commands>true</use_force_commands>
             <sub_topic>joint/hip_joint/0/cmd_pos</sub_topic>
-            <p_gain>200.0</p_gain>
-            <i_gain>0.0</i_gain>
-            <d_gain>50.0</d_gain>
-            <i_max>1</i_max>
-            <i_min>-1</i_min>
+            <p_gain>5000.0</p_gain>
+            <i_gain>1.0</i_gain>
+            <d_gain>500.0</d_gain>
+            <i_max>100</i_max>
+            <i_min>-100</i_min>
             <cmd_max>100</cmd_max>
             <cmd_min>-100</cmd_min>
             <cmd_offset>0.0</cmd_offset>
-            <!-- <initial_position>-0.3</initial_position> -->
         </plugin>
         <plugin
@@ -24,13 +23,12 @@
             <use_force_commands>true</use_force_commands>
             <sub_topic>joint/knee_joint/0/cmd_pos</sub_topic>
-            <p_gain>100.0</p_gain>
-            <i_gain>0.0</i_gain>
-            <d_gain>10.0</d_gain>
-            <i_max>1</i_max>
-            <i_min>-1</i_min>
+            <p_gain>5000.0</p_gain>
+            <i_gain>1.0</i_gain>
+            <d_gain>500.0</d_gain>
+            <i_max>100</i_max>
+            <i_min>-100</i_min>
             <cmd_max>100</cmd_max>
             <cmd_min>-100</cmd_min>
             <cmd_offset>0.0</cmd_offset>
-            <!-- <initial_position>0.6</initial_position> -->
         </plugin>
     </gazebo>

File: ros2_ws/src/robot_description/description/robot.urdf.xacro (robot description, xacro)
@@ -6,4 +6,5 @@
     <xacro:property name="L1_length" default="0.3"/>
     <xacro:property name="L2_length" default="0.25"/>
+    <xacro:property name="max_torque" default="20.1"/>
     <link name="world">
     </link>
@@ -14,5 +15,5 @@
         <axis xyz="0 0 1" />
         <limit effort="0" lower="-10" upper="10" velocity="100.0" />
-        <dynamics damping="0.0" friction="0.1" />
+        <dynamics damping="0.0" friction="0.0" />
     </joint>
     <link name="base_link">
@@ -27,5 +28,5 @@
         <origin xyz="0 0 0" rpy="${pi/2} -${pi/2} 0" />
         <axis xyz="0 0 1" />
-        <limit effort="10.5" lower="-${pi}" upper="${pi}" velocity="62.9" />
+        <limit effort="${max_torque}" lower="-${pi}" upper="${pi}" velocity="62.9" />
         <dynamics damping="0.1" friction="0.1" />
     </joint>
@@ -48,5 +49,5 @@
         <inertial>
             <origin xyz="0 0 0" rpy="0 0 0" />
-            <mass value="1" />
+            <mass value="0.6" />
             <inertia ixx="0.01" ixy="0" ixz="0" iyy="0.01" iyz="0" izz="0.01" />
         </inertial>
@@ -57,5 +58,5 @@
         <origin xyz="${-L1_length} 0 0" rpy="0 0 0" />
         <axis xyz="0 0 1" />
-        <limit effort="10.5" lower="-${pi}" upper="${pi}" velocity="62.9" />
+        <limit effort="${max_torque}" lower="-${pi}" upper="${pi}" velocity="62.9" />
         <dynamics damping="0.1" friction="0.1" />
     </joint>
@@ -78,5 +79,5 @@
         <inertial>
             <origin xyz="0 0 0" rpy="0 0 0" />
-            <mass value="1" />
+            <mass value="0.1" />
             <inertia ixx="0.01" ixy="0" ixz="0" iyy="0.01" iyz="0" izz="0.01" />
         </inertial>
@@ -84,6 +85,6 @@
     <!-- This has to be a revolute joint for some dumb reason -->
     <!-- Can also change this manually in the sdf to a fixed joint -->
-    <!-- <joint name="contact_joint" type="fixed"> -->
-    <joint name="contact_joint" type="revolute">
+    <joint name="contact_joint" type="fixed">
+    <!-- <joint name="contact_joint" type="revolute"> -->
         <parent link="knee_link" />
         <child link="foot_link" />
@@ -91,5 +92,5 @@
         <axis xyz="0 0 1" />
         <limit effort="1e-5" lower="0" upper="0" velocity="1e-5" />
-        <dynamics damping="0.1" friction="0.1" />
+        <dynamics damping="0.0" friction="0.0" />
     </joint>
     <link name="foot_link">
@@ -100,8 +101,7 @@
         </visual>
         <!-- Something is wrong with the urdf/xacro/sdf conversion.
-         This collision name changes when the sim is launched.
-         To change this, export the entire world after you launch gazebo as an sdf file
-         and then go in manually and change the name back -->
-        <collision name="foot_collision">
+         This collision name changes when the sim is launched. -->
+        <!-- <collision name="foot_collision"> -->
+        <collision>
             <geometry>
                 <sphere radius="0.05" />

File: ros2_ws/src/robot_description/description/simulation.xacro (robot description, xacro)
@@ -1,20 +1,20 @@
 <?xml version="1.0"?>
 <robot xmlns:xacro="http://www.ros.org/wiki/xacro">
-    <link name="imu_link"></link>
-    <joint name="imu_joint" type="fixed">
-        <parent link="base_link" />
-        <child link="imu_link" />
-        <origin xyz="0 0 0" rpy="0 0 0" />
-    </joint>
-    <gazebo reference="imu_link">
-        <sensor name="imu" type="imu">
-            <always_on>true</always_on>
-            <update_rate>100.0</update_rate>
-            <visualize>true</visualize>
-            <topic>/model/robot/sensors/imu</topic>
-            <gz_frame_id>imu_link</gz_frame_id>
-            <imu>
-                <!-- noise statistics -->
-                <!-- <angular_velocity>
+  <link name="imu_link"></link>
+  <joint name="imu_joint" type="fixed">
+    <parent link="base_link" />
+    <child link="imu_link" />
+    <origin xyz="0 0 0" rpy="0 0 0" />
+  </joint>
+  <gazebo reference="imu_link">
+    <sensor name="imu" type="imu">
+      <always_on>true</always_on>
+      <update_rate>100.0</update_rate>
+      <visualize>true</visualize>
+      <topic>/model/robot/sensors/imu</topic>
+      <gz_frame_id>imu_link</gz_frame_id>
+      <imu>
+        <!-- noise statistics -->
+        <!-- <angular_velocity>
                 <x>
                     <noise type="gaussian">
@@ -86,32 +86,32 @@
                   </z>
                 </linear_acceleration> -->
-                <orientation_reference_frame>
-                  <localization>ENU</localization>
-                </orientation_reference_frame>
-            </imu>
-        </sensor>
-    </gazebo>
-    <gazebo>
-        <plugin
-            filename="gz-sim-joint-state-publisher-system"
-            name="gz::sim::systems::JointStatePublisher">
-            <topic>model/robot/joint_states</topic>
-            <joint_name>hip_joint</joint_name>
-            <joint_name>knee_joint</joint_name>
-        </plugin>
-        <plugin
-            filename="gz-sim-contact-system"
-            name="gz::sim::systems::Contact">
-        </plugin>
-    </gazebo>
-    <gazebo reference="foot_link">
-        <sensor name='foot_contact' type='contact'>
-            <always_on>true</always_on>
-            <update_rate>100.0</update_rate>
-            <contact>
-                <collision>foot_link_collision</collision>
-                <topic>/model/robot/sensors/contact</topic>
-            </contact>
-        </sensor>
-    </gazebo>
+        <orientation_reference_frame>
+          <localization>ENU</localization>
+        </orientation_reference_frame>
+      </imu>
+    </sensor>
+  </gazebo>
+  <gazebo reference="contact_joint">
+    <preserveFixedJoint>True</preserveFixedJoint>
+  </gazebo>
+  <gazebo>
+    <plugin
+      filename="gz-sim-joint-state-publisher-system"
+      name="gz::sim::systems::JointStatePublisher">
+      <topic>model/robot/joint_states</topic>
+      <joint_name>hip_joint</joint_name>
+      <joint_name>knee_joint</joint_name>
+    </plugin>
+  </gazebo>
+  <gazebo reference="foot_link">
+    <sensor name='foot_contact' type='contact'>
+      <always_on>true</always_on>
+      <update_rate>500.0</update_rate>
+      <contact>
+        <collision>foot_link_collision</collision>
+        <!-- <collision>foot_link_fixed_joint_lump__foot_collision_collision</collision> -->
+        <topic>/model/robot/sensors/contact</topic>
+      </contact>
+    </sensor>
+  </gazebo>
 </robot>

Commit message: update readme

File: ros2_ws/src/robot_description/description/position_control.xacro (robot description, xacro)
@@ -6,5 +6,4 @@
             name="gz::sim::systems::JointPositionController">
             <joint_name>hip_joint</joint_name>
-            <use_force_commands>true</use_force_commands>
             <sub_topic>joint/hip_joint/0/cmd_pos</sub_topic>
             <p_gain>5000.0</p_gain>
@@ -13,6 +12,6 @@
             <i_max>100</i_max>
             <i_min>-100</i_min>
-            <cmd_max>100</cmd_max>
-            <cmd_min>-100</cmd_min>
+            <cmd_max>${max_torque}</cmd_max>
+            <cmd_min>${-max_torque}</cmd_min>
             <cmd_offset>0.0</cmd_offset>
         </plugin>
@@ -21,5 +20,4 @@
             name="gz::sim::systems::JointPositionController">
             <joint_name>knee_joint</joint_name>
-            <use_force_commands>true</use_force_commands>
             <sub_topic>joint/knee_joint/0/cmd_pos</sub_topic>
             <p_gain>5000.0</p_gain>
@@ -28,6 +26,6 @@
             <i_max>100</i_max>
             <i_min>-100</i_min>
-            <cmd_max>100</cmd_max>
-            <cmd_min>-100</cmd_min>
+            <cmd_max>${max_torque}</cmd_max>
+            <cmd_min>${-max_torque}</cmd_min>
             <cmd_offset>0.0</cmd_offset>
         </plugin>

File: ros2_ws/src/robot_description/description/robot.urdf.xacro (robot description, xacro)
@@ -26,5 +26,5 @@
         <parent link="base_link" />
         <child link="hip_link" />
-        <origin xyz="0 0 0" rpy="${pi/2} -${pi/2} 0" />
+        <origin xyz="0 0 0" rpy="${pi/2} ${pi/2} 0" />
         <axis xyz="0 0 1" />
         <limit effort="${max_torque}" lower="-${pi}" upper="${pi}" velocity="62.9" />
@@ -33,5 +33,5 @@
     <link name="hip_link">
         <visual>
-            <origin xyz="${-L1_length/2} 0 0" rpy="0 0 0" />
+            <origin xyz="${L1_length/2} 0 0" rpy="0 0 0" />
             <geometry>
                 <box size="${L1_length} 0.05 0.02" />
@@ -56,5 +56,5 @@
         <parent link="hip_link" />
         <child link="knee_link" />
-        <origin xyz="${-L1_length} 0 0" rpy="0 0 0" />
+        <origin xyz="${L1_length} 0 0" rpy="0 0 0" />
         <axis xyz="0 0 1" />
         <limit effort="${max_torque}" lower="-${pi}" upper="${pi}" velocity="62.9" />
@@ -63,5 +63,5 @@
     <link name="knee_link">
         <visual>
-            <origin xyz="${-L2_length/2} 0 0" rpy="0 0 0" />
+            <origin xyz="${L2_length/2} 0 0" rpy="0 0 0" />
             <geometry>
                 <box size="${L2_length} 0.05 0.02" />
@@ -89,5 +89,5 @@
         <parent link="knee_link" />
         <child link="foot_link" />
-        <origin xyz="${-L2_length} 0 0" rpy="0 0 0" />
+        <origin xyz="${L2_length} 0 0" rpy="0 0 0" />
         <axis xyz="0 0 1" />
         <limit effort="1e-5" lower="0" upper="0" velocity="1e-5" />

File: ros2_ws/src/robot_description/description/torque_control.xacro (robot description, xacro)
@@ -14,6 +14,6 @@
             <i_max>1</i_max>
             <i_min>-1</i_min>
-            <cmd_max>100</cmd_max>
-            <cmd_min>-100</cmd_min>
+            <cmd_max>${max_torque}</cmd_max>
+            <cmd_min>${-max_torque}</cmd_min>
             <cmd_offset>0.0</cmd_offset>
         </plugin>
@@ -30,6 +30,6 @@
             <i_max>1</i_max>
             <i_min>-1</i_min>
-            <cmd_max>100</cmd_max>
-            <cmd_min>-100</cmd_min>
+            <cmd_max>${max_torque}</cmd_max>
+            <cmd_min>${-max_torque}</cmd_min>
             <cmd_offset>0.0</cmd_offset>
         </plugin>

Commit message: dynamics eqn

File: ros2_ws/src/robot_description/description/position_control.xacro (robot description, xacro)
@@ -7,7 +7,7 @@
             <joint_name>hip_joint</joint_name>
             <sub_topic>joint/hip_joint/0/cmd_pos</sub_topic>
-            <p_gain>5000.0</p_gain>
-            <i_gain>1.0</i_gain>
-            <d_gain>500.0</d_gain>
+            <p_gain>150.0</p_gain>
+            <i_gain>0.0</i_gain>
+            <d_gain>15.0</d_gain>
             <i_max>100</i_max>
             <i_min>-100</i_min>
@@ -21,7 +21,7 @@
             <joint_name>knee_joint</joint_name>
             <sub_topic>joint/knee_joint/0/cmd_pos</sub_topic>
-            <p_gain>5000.0</p_gain>
-            <i_gain>1.0</i_gain>
-            <d_gain>500.0</d_gain>
+            <p_gain>100.0</p_gain>
+            <i_gain>0.0</i_gain>
+            <d_gain>10.0</d_gain>
             <i_max>100</i_max>
             <i_min>-100</i_min>

File: ros2_ws/src/robot_description/description/robot.urdf.xacro (robot description, xacro)
@@ -4,6 +4,8 @@
     <xacro:arg name="torque_control" default="false" />
     <xacro:arg name="position_control" default="false" />
-    <xacro:property name="L1_length" default="0.093732"/>
-    <xacro:property name="L2_length" default="0.125"/>
+    <xacro:property name="L1_length" default="0.3"/>
+    <!-- <xacro:property name="L1_length" default="0.093732"/> -->
+    <xacro:property name="L2_length" default="0.25"/>
+    <!-- <xacro:property name="L2_length" default="0.125"/> -->
     <xacro:property name="max_torque" default="20.1"/>
     <link name="world">
@@ -19,4 +21,5 @@
     <link name="base_link">
         <inertial>
+            <origin xyz="0 0 0" rpy="0 0 0" />
             <mass value="0.01" />
             <inertia ixx="0.01" ixy="0" ixz="0" iyy="0.01" iyz="0" izz="0.01" />
@@ -28,15 +31,15 @@
         <origin xyz="0 0 0" rpy="${pi/2} ${pi/2} 0" />
         <axis xyz="0 0 1" />
-        <limit effort="${max_torque}" lower="-${pi}" upper="${pi}" velocity="62.9" />
+        <limit effort="${max_torque}" lower="-${pi}" upper="${pi}" velocity="31.67" />
         <dynamics damping="0.1" friction="0.1" />
     </joint>
     <link name="hip_link">
         <visual>
-            <!-- <origin xyz="${L1_length/2} 0 0" rpy="0 0 0" /> -->
+            <origin xyz="${L1_length/2} 0 0" rpy="0 0 0" />
             <geometry>
-                <mesh filename="file://$(find robot_description)/meshes/hip.stl"/>
+                <!-- <mesh filename="file://$(find robot_description)/meshes/hip.stl"/> -->
                 <!-- for preview -->
                 <!-- <mesh filename="../meshes/hip.stl"/> -->
-                <!-- <box size="${L1_length} 0.05 0.02" /> -->
+                <box size="${L1_length} 0.05 0.02" />
             </geometry>
             <material name="blue">
@@ -61,15 +64,15 @@
         <origin xyz="${L1_length} 0 0" rpy="0 0 0" />
         <axis xyz="0 0 1" />
-        <limit effort="${max_torque}" lower="-${pi}" upper="${pi}" velocity="62.9" />
+        <limit effort="${max_torque}" lower="-${pi}" upper="${pi}" velocity="31.67" />
         <dynamics damping="0.1" friction="0.1" />
     </joint>
     <link name="knee_link">
         <visual>
-            <!-- <origin xyz="${L2_length/2} 0 0" rpy="0 0 0" /> -->
+            <origin xyz="${L2_length/2} 0 0" rpy="0 0 0" />
             <geometry>
-                <mesh filename="file://$(find robot_description)/meshes/tibia.stl"/>
+                <!-- <mesh filename="file://$(find robot_description)/meshes/tibia.stl"/> -->
                 <!-- for preview -->
                 <!-- <mesh filename="../meshes/tibia.stl"/> -->
-                <!-- <box size="${L2_length} 0.05 0.02" /> -->
+                <box size="${L2_length} 0.05 0.02" />
             </geometry>
             <material name="green">
@@ -103,5 +106,5 @@
         <visual>
             <geometry>
-                <sphere radius="0.01" />
+                <sphere radius="0.05" />
             </geometry>
         </visual>
@@ -111,5 +114,5 @@
         <collision>
             <geometry>
-                <sphere radius="0.01" />
+                <sphere radius="0.05" />
             </geometry>
         </collision>

File: ros2_ws/src/robot_description/description/simulation.xacro (robot description, xacro)
@@ -10,5 +10,5 @@
     <sensor name="imu" type="imu">
       <always_on>true</always_on>
-      <update_rate>100.0</update_rate>
+      <update_rate>500.0</update_rate>
       <visualize>true</visualize>
       <topic>/model/robot/sensors/imu</topic>
@@ -87,5 +87,5 @@
                 </linear_acceleration> -->
         <orientation_reference_frame>
-          <localization>ENU</localization>
+          <localization>NWU</localization>
         </orientation_reference_frame>
       </imu>

File: ros2_ws/src/robot_description/description/torque_control.xacro (robot description, xacro)
@@ -9,7 +9,7 @@
             <inital_velocity>0</inital_velocity>
             <sub_topic>joint/hip_joint/0/cmd_torque</sub_topic>
-            <p_gain>1.0</p_gain>
+            <p_gain>150.0</p_gain>
             <i_gain>0.0</i_gain>
-            <d_gain>0.1</d_gain>
+            <d_gain>15.0</d_gain>
             <i_max>1</i_max>
             <i_min>-1</i_min>
@@ -25,7 +25,7 @@
             <inital_velocity>0</inital_velocity>
             <sub_topic>joint/knee_joint/0/cmd_torque</sub_topic>
-            <p_gain>1.0</p_gain>
+            <p_gain>100.0</p_gain>
             <i_gain>0.0</i_gain>
-            <d_gain>0.1</d_gain>
+            <d_gain>10.0</d_gain>
             <i_max>1</i_max>
             <i_min>-1</i_min>
