Commit message: urdf parser and fk

File: ros2_ws/src/robot_description/description/robot.urdf.xacro (robot description, xacro)
@@ -42,4 +42,5 @@
         </collision>
         <inertial>
+            <origin xyz="0 0 0" rpy="0 0 0" />
             <mass value="1" />
             <inertia ixx="0.01" ixy="0" ixz="0" iyy="0.01" iyz="0" izz="0.01" />
@@ -71,4 +72,5 @@
         </collision>
         <inertial>
+            <origin xyz="0 0 0" rpy="0 0 0" />
             <mass value="1" />
             <inertia ixx="0.01" ixy="0" ixz="0" iyy="0.01" iyz="0" izz="0.01" />
@@ -82,5 +84,10 @@
     </joint>
     <link name="foot">
-        <collision>
+        <visual>
+            <geometry>
+                <sphere radius="0.05" />
+            </geometry>
+        </visual>
+        <collision name="foot_collision">
             <origin xyz="0 0 0" rpy="0 0 0" />
             <geometry>
@@ -89,4 +96,4 @@
         </collision>
     </link>
-    <xacro:include filename="$(find robot_description)/description/simulation.xacro" />
+    <!-- <xacro:include filename="$(find robot_description)/description/simulation.xacro" /> -->
 </robot>

File: ros2_ws/src/robot_description/description/simulation.xacro (robot description, xacro)
@@ -3,10 +3,9 @@
     <gazebo>
         <plugin
-            filename="gz-sim-contact-system"
-            name="gz::sim::systems::Contact">
-        </plugin>
-        <plugin
             filename="gz-sim-joint-state-publisher-system"
             name="gz::sim::systems::JointStatePublisher">
+            <topic>model/robot/joint_states</topic>
+            <joint_name>hip_joint</joint_name>
+            <joint_name>knee_joint</joint_name>
         </plugin>
         <plugin
@@ -17,4 +16,12 @@
             <inital_velocity>0</inital_velocity>
             <sub_topic>joint/hip_joint/0/cmd_torque</sub_topic>
+            <p_gain>1.0</p_gain>
+            <i_gain>0.0</i_gain>
+            <d_gain>0.1</d_gain>
+            <i_max>1</i_max>
+            <i_min>-1</i_min>
+            <cmd_max>100</cmd_max>
+            <cmd_min>-100</cmd_min>
+            <cmd_offset>0.0</cmd_offset>
         </plugin>
         <plugin
@@ -25,14 +32,30 @@
             <inital_velocity>0</inital_velocity>
             <sub_topic>joint/knee_joint/0/cmd_torque</sub_topic>
+            <p_gain>1.0</p_gain>
+            <i_gain>0.0</i_gain>
+            <d_gain>0.1</d_gain>
+            <i_max>1</i_max>
+            <i_min>-1</i_min>
+            <cmd_max>100</cmd_max>
+            <cmd_min>-100</cmd_min>
+            <cmd_offset>0.0</cmd_offset>
         </plugin>
-        <sensor name="contact" type="contact">
+    </gazebo>
+    <gazebo reference="foot">
+        <sensor name="contact_sensor" type="contact">
             <always_on>true</always_on>
             <update_rate>10.0</update_rate>
             <visualize>true</visualize>
             <contact>
-                <collision>foot</collision>
-                <!-- <topic></topic> -->
+                <collision>foot_collision</collision>
+                <topic>/model/robot/contact</topic>
             </contact>
         </sensor>
+        <plugin filename="gz-sim-touchplugin-system"
+            name="gz::sim::systems::TouchPlugin">
+            <target>collision</target>
+            <time>0.001</time>
+            <enabled>true</enabled>
+        </plugin>
     </gazebo>
 </robot>

Commit message: finally got contact sensor working, this whole ros2 gz sim pipeline is sooo stupid

File: ros2_ws/src/robot_description/description/robot.urdf.xacro (robot description, xacro)
@@ -1,4 +1,9 @@
 <?xml version="1.0"?>
 <robot xmlns:xacro="http://www.ros.org/wiki/xacro" name="robot">
+    <xacro:arg name="use_sim_time" default="false" />
+    <xacro:arg name="torque_control" default="false" />
+    <xacro:arg name="position_control" default="false" />
+    <xacro:property name="L1_length" default="0.3"/>
+    <xacro:property name="L2_length" default="0.25"/>
     <link name="world">
     </link>
@@ -6,7 +11,7 @@
         <parent link="world" />
         <child link="base_link" />
-        <origin xyz="0 0 0" rpy="0 0 0" />
+        <origin xyz="0 0 1.0" rpy="0 0 0" />
         <axis xyz="0 0 1" />
-        <limit effort="0" lower="0" upper="2" velocity="100.0" />
+        <limit effort="0" lower="-10" upper="10" velocity="100.0" />
         <dynamics damping="0.0" friction="0.1" />
     </joint>
@@ -19,5 +24,5 @@
     <joint name="hip_joint" type="revolute">
         <parent link="base_link" />
-        <child link="hip" />
+        <child link="hip_link" />
         <origin xyz="0 0 0" rpy="${pi/2} -${pi/2} 0" />
         <axis xyz="0 0 1" />
@@ -25,9 +30,9 @@
         <dynamics damping="0.1" friction="0.1" />
     </joint>
-    <link name="hip">
+    <link name="hip_link">
         <visual>
-            <origin xyz="-0.15 0 0" rpy="0 0 0" />
+            <origin xyz="${-L1_length/2} 0 0" rpy="0 0 0" />
             <geometry>
-                <box size="0.3 0.05 0.02" />
+                <box size="${L1_length} 0.05 0.02" />
             </geometry>
             <material name="blue">
@@ -36,7 +41,7 @@
         </visual>
         <collision>
-            <origin xyz="-0.15 0 0" rpy="0 0 0" />
+            <origin xyz="${-L1_length/2} 0 0" rpy="0 0 0" />
             <geometry>
-                <box size="0.3 0.05 0.02" />
+                <box size="${L1_length} 0.05 0.02" />
             </geometry>
         </collision>
@@ -48,16 +53,16 @@
     </link>
     <joint name="knee_joint" type="revolute">
-        <parent link="hip" />
-        <child link="knee" />
-        <origin xyz="-0.3 0 0" rpy="0 0 0" />
+        <parent link="hip_link" />
+        <child link="knee_link" />
+        <origin xyz="${-L1_length} 0 0" rpy="0 0 0" />
         <axis xyz="0 0 1" />
         <limit effort="10.5" lower="-${pi}" upper="${pi}" velocity="62.9" />
         <dynamics damping="0.1" friction="0.1" />
     </joint>
-    <link name="knee">
+    <link name="knee_link">
         <visual>
-            <origin xyz="-0.125 0 0" rpy="0 0 0" />
+            <origin xyz="${-L2_length/2} 0 0" rpy="0 0 0" />
             <geometry>
-                <box size="0.25 0.05 0.02" />
+                <box size="${L2_length} 0.05 0.02" />
             </geometry>
             <material name="green">
@@ -66,7 +71,7 @@
         </visual>
         <collision>
-            <origin xyz="-0.125 0 0" rpy="0 0 0" />
+            <origin xyz="${-L2_length/2} 0 0" rpy="0 0 0" />
             <geometry>
-                <box size="0.25 0.05 0.02" />
+                <box size="${L2_length} 0.05 0.02" />
             </geometry>
         </collision>
@@ -77,11 +82,13 @@
         </inertial>
     </link>
-    <joint name="contact_joint" type="fixed">
-        <parent link="knee" />
-        <child link="foot" />
-        <origin xyz="-0.25 0 0" rpy="0 0 0" />
+    <!-- This has to be a revolute joint for some dumb reason -->
+    <joint name="contact_joint" type="revolute">
+        <parent link="knee_link" />
+        <child link="foot_link" />
+        <origin xyz="${-L2_length} 0 0" rpy="0 0 0" />
         <axis xyz="0 0 1" />
+        <limit effort="1e-5" lower="0" upper="0" velocity="1e-5" />
     </joint>
-    <link name="foot">
+    <link name="foot_link">
         <visual>
             <geometry>
@@ -89,11 +96,26 @@
             </geometry>
         </visual>
+        <!-- Something is wrong with the urdf/xacro/sdf conversion.
+         This collision name changes when the sim is launched.
+         To change this, export the entire world after you launch gazebo as an sdf file
+         and then go in manually and change the name back -->
         <collision name="foot_collision">
-            <origin xyz="0 0 0" rpy="0 0 0" />
             <geometry>
                 <sphere radius="0.05" />
             </geometry>
         </collision>
+        <inertial>
+            <mass value="0.01" />
+            <inertia ixx="0.01" ixy="0" ixz="0" iyy="0.01" iyz="0" izz="0.01" />
+        </inertial>
     </link>
-    <!-- <xacro:include filename="$(find robot_description)/description/simulation.xacro" /> -->
+    <xacro:if value="$(arg use_sim_time)">
+        <xacro:include filename="$(find robot_description)/description/simulation.xacro" />
+        <xacro:if value="$(arg torque_control)">
+            <xacro:include filename="$(find robot_description)/description/torque_control.xacro" />
+        </xacro:if>
+        <xacro:if value="$(arg position_control)">
+            <xacro:include filename="$(find robot_description)/description/position_control.xacro" />
+        </xacro:if>
+    </xacro:if>
 </robot>

File: ros2_ws/src/robot_description/description/simulation.xacro (robot description, xacro)
@@ -1,4 +1,95 @@
 <?xml version="1.0"?>
-<robot xmlns:xacro="http://www.ros.org/wiki/xacro" name="robot">
+<robot xmlns:xacro="http://www.ros.org/wiki/xacro">
+    <link name="imu_link"></link>
+    <joint name="imu_joint" type="fixed">
+        <parent link="base_link" />
+        <child link="imu_link" />
+        <origin xyz="0 0 0" rpy="0 0 0" />
+    </joint>
+    <gazebo reference="imu_link">
+        <sensor name="imu" type="imu">
+            <always_on>true</always_on>
+            <update_rate>100.0</update_rate>
+            <visualize>true</visualize>
+            <topic>/model/robot/sensors/imu</topic>
+            <gz_frame_id>imu_link</gz_frame_id>
+            <imu>
+                <!-- noise statistics -->
+                <!-- <angular_velocity>
+                <x>
+                    <noise type="gaussian">
+                      <mean>0</mean>
+                      <stddev>0.009</stddev>
+                      <bias_mean>0.00075</bias_mean>
+                      <bias_stddev>0.005</bias_stddev>
+                      <dynamic_bias_stddev>0.00002</dynamic_bias_stddev>
+                      <dynamic_bias_correlation_time>400.0</dynamic_bias_correlation_time>
+                      <precision>0.00025</precision>
+                    </noise>
+                  </x>
+                  <y>
+                    <noise type="gaussian">
+                      <mean>0</mean>
+                      <stddev>0.009</stddev>
+                      <bias_mean>0.00075</bias_mean>
+                      <bias_stddev>0.005</bias_stddev>
+                      <dynamic_bias_stddev>0.00002</dynamic_bias_stddev>
+                      <dynamic_bias_correlation_time>400.0</dynamic_bias_correlation_time>
+                      <precision>0.00025</precision>
+                    </noise>
+                  </y>
+                  <z>
+                    <noise type="gaussian">
+                      <mean>0</mean>
+                      <stddev>0.009</stddev>
+                      <bias_mean>0.00075</bias_mean>
+                      <bias_stddev>0.005</bias_stddev>
+                      <dynamic_bias_stddev>0.00002</dynamic_bias_stddev>
+                      <dynamic_bias_correlation_time>400.0</dynamic_bias_correlation_time>
+                      <precision>0.00025</precision>
+                    </noise>
+                  </z>
+                </angular_velocity>
+                <linear_acceleration>
+                  <x>
+                    <noise type="gaussian">
+                      <mean>0</mean>
+                      <stddev>0.021</stddev>
+                      <bias_mean>0.05</bias_mean>
+                      <bias_stddev>0.0075</bias_stddev>
+                      <dynamic_bias_stddev>0.000375</dynamic_bias_stddev>
+                      <dynamic_bias_correlation_time>175.0</dynamic_bias_correlation_time>
+                      <precision>0.005</precision>
+                    </noise>
+                  </x>
+                  <y>
+                    <noise type="gaussian">
+                      <mean>0</mean>
+                      <stddev>0.021</stddev>
+                      <bias_mean>0.05</bias_mean>
+                      <bias_stddev>0.0075</bias_stddev>
+                      <dynamic_bias_stddev>0.000375</dynamic_bias_stddev>
+                      <dynamic_bias_correlation_time>175.0</dynamic_bias_correlation_time>
+                      <precision>0.005</precision>
+                    </noise>
+                  </y>
+                  <z>
+                    <noise type="gaussian">
+                      <mean>0</mean>
+                      <stddev>0.021</stddev>
+                      <bias_mean>0.05</bias_mean>
+                      <bias_stddev>0.0075</bias_stddev>
+                      <dynamic_bias_stddev>0.000375</dynamic_bias_stddev>
+                      <dynamic_bias_correlation_time>175.0</dynamic_bias_correlation_time>
+                      <precision>0.005</precision>
+                    </noise>
+                  </z>
+                </linear_acceleration> -->
+                <orientation_reference_frame>
+                  <localization>ENU</localization>
+                </orientation_reference_frame>
+            </imu>
+        </sensor>
+    </gazebo>
     <gazebo>
         <plugin
@@ -10,52 +101,17 @@
         </plugin>
         <plugin
-            filename="gz-sim-joint-controller-system"
-            name="gz::sim::systems::JointController">
-            <joint_name>hip_joint</joint_name>
-            <use_force_commands>true</use_force_commands>
-            <inital_velocity>0</inital_velocity>
-            <sub_topic>joint/hip_joint/0/cmd_torque</sub_topic>
-            <p_gain>1.0</p_gain>
-            <i_gain>0.0</i_gain>
-            <d_gain>0.1</d_gain>
-            <i_max>1</i_max>
-            <i_min>-1</i_min>
-            <cmd_max>100</cmd_max>
-            <cmd_min>-100</cmd_min>
-            <cmd_offset>0.0</cmd_offset>
-        </plugin>
-        <plugin
-            filename="gz-sim-joint-controller-system"
-            name="gz::sim::systems::JointController">
-            <joint_name>knee_joint</joint_name>
-            <use_force_commands>true</use_force_commands>
-            <inital_velocity>0</inital_velocity>
-            <sub_topic>joint/knee_joint/0/cmd_torque</sub_topic>
-            <p_gain>1.0</p_gain>
-            <i_gain>0.0</i_gain>
-            <d_gain>0.1</d_gain>
-            <i_max>1</i_max>
-            <i_min>-1</i_min>
-            <cmd_max>100</cmd_max>
-            <cmd_min>-100</cmd_min>
-            <cmd_offset>0.0</cmd_offset>
+            filename="gz-sim-contact-system"
+            name="gz::sim::systems::Contact">
         </plugin>
     </gazebo>
-    <gazebo reference="foot">
-        <sensor name="contact_sensor" type="contact">
+    <gazebo reference="foot_link">
+        <sensor name='foot_contact' type='contact'>
             <always_on>true</always_on>
-            <update_rate>10.0</update_rate>
-            <visualize>true</visualize>
+            <update_rate>100.0</update_rate>
             <contact>
                 <collision>foot_collision</collision>
-                <topic>/model/robot/contact</topic>
+                <topic>/model/robot/sensors/contact</topic>
             </contact>
         </sensor>
-        <plugin filename="gz-sim-touchplugin-system"
-            name="gz::sim::systems::TouchPlugin">
-            <target>collision</target>
-            <time>0.001</time>
-            <enabled>true</enabled>
-        </plugin>
     </gazebo>
 </robot>

Commit message: stupid urdf-sdf converter is straight up broken

File: ros2_ws/src/robot_description/description/robot.urdf.xacro (robot description, xacro)
@@ -83,4 +83,5 @@
     </link>
     <!-- This has to be a revolute joint for some dumb reason -->
+    <!-- Can also change this manually in the sdf to a fixed joint -->
     <joint name="contact_joint" type="revolute">
         <parent link="knee_link" />

File: ros2_ws/src/robot_description/description/simulation.xacro (robot description, xacro)
@@ -110,5 +110,5 @@
             <update_rate>100.0</update_rate>
             <contact>
-                <collision>foot_collision</collision>
+                <collision>foot_link_collision</collision>
                 <topic>/model/robot/sensors/contact</topic>
             </contact>

Commit message: add meshes to prevent build error, fix ik, edit readme for venv setup

File: ros2_ws/src/robot_description/description/robot.urdf.xacro (robot description, xacro)
@@ -4,6 +4,6 @@
     <xacro:arg name="torque_control" default="false" />
     <xacro:arg name="position_control" default="false" />
-    <xacro:property name="L1_length" default="0.3"/>
-    <xacro:property name="L2_length" default="0.25"/>
+    <xacro:property name="L1_length" default="0.093732"/>
+    <xacro:property name="L2_length" default="0.125"/>
     <xacro:property name="max_torque" default="20.1"/>
     <link name="world">
@@ -33,7 +33,8 @@
     <link name="hip_link">
         <visual>
-            <origin xyz="${L1_length/2} 0 0" rpy="0 0 0" />
+            <!-- <origin xyz="${L1_length/2} 0 0" rpy="0 0 0" /> -->
             <geometry>
-                <box size="${L1_length} 0.05 0.02" />
+                <mesh filename="file://$(find robot_description)/meshes/hip.stl"/>
+                <!-- <box size="${L1_length} 0.05 0.02" /> -->
             </geometry>
             <material name="blue">
@@ -63,7 +64,8 @@
     <link name="knee_link">
         <visual>
-            <origin xyz="${L2_length/2} 0 0" rpy="0 0 0" />
+            <!-- <origin xyz="${L2_length/2} 0 0" rpy="0 0 0" /> -->
             <geometry>
-                <box size="${L2_length} 0.05 0.02" />
+                <mesh filename="file://$(find robot_description)/meshes/tibia.stl"/>
+                <!-- <box size="${L2_length} 0.05 0.02" /> -->
             </geometry>
             <material name="green">
@@ -97,5 +99,5 @@
         <visual>
             <geometry>
-                <sphere radius="0.05" />
+                <sphere radius="0.01" />
             </geometry>
         </visual>
@@ -105,5 +107,5 @@
         <collision>
             <geometry>
-                <sphere radius="0.05" />
+                <sphere radius="0.01" />
             </geometry>
         </collision>

Commit message: add preview path for urdf

File: ros2_ws/src/robot_description/description/robot.urdf.xacro (robot description, xacro)
@@ -36,4 +36,6 @@
             <geometry>
                 <mesh filename="file://$(find robot_description)/meshes/hip.stl"/>
+                <!-- for preview -->
+                <!-- <mesh filename="../meshes/hip.stl"/> -->
                 <!-- <box size="${L1_length} 0.05 0.02" /> -->
             </geometry>
@@ -43,5 +45,5 @@
         </visual>
         <collision>
-            <origin xyz="${-L1_length/2} 0 0" rpy="0 0 0" />
+            <origin xyz="${L1_length/2} 0 0" rpy="0 0 0" />
             <geometry>
                 <box size="${L1_length} 0.05 0.02" />
@@ -67,4 +69,6 @@
             <geometry>
                 <mesh filename="file://$(find robot_description)/meshes/tibia.stl"/>
+                <!-- for preview -->
+                <!-- <mesh filename="../meshes/tibia.stl"/> -->
                 <!-- <box size="${L2_length} 0.05 0.02" /> -->
             </geometry>
@@ -74,7 +78,7 @@
         </visual>
         <collision>
-            <origin xyz="${-L2_length/2} 0 0" rpy="0 0 0" />
+            <origin xyz="${L2_length/2} 0 0" rpy="0 0 0" />
             <geometry>
-                <box size="${L2_length} 0.05 0.02" />
+                <box size="${L2_length} 0.01 0.04" />
             </geometry>
         </collision>

Commit message: wrote active compliance, but something is wrong

File: ros2_ws/src/robot_description/description/robot.urdf.xacro (robot description, xacro)
@@ -31,6 +31,6 @@
         <origin xyz="0 0 0" rpy="${pi/2} ${pi/2} 0" />
         <axis xyz="0 0 1" />
-        <limit effort="${max_torque}" lower="-${pi}" upper="${pi}" velocity="31.67" />
-        <dynamics damping="0.1" friction="0.1" />
+        <limit effort="${max_torque}" lower="-${pi/2}" upper="0" velocity="31.67" />
+        <dynamics damping="0.01" friction="0.01" />
     </joint>
     <link name="hip_link">
@@ -64,6 +64,6 @@
         <origin xyz="${L1_length} 0 0" rpy="0 0 0" />
         <axis xyz="0 0 1" />
-        <limit effort="${max_torque}" lower="-${pi}" upper="${pi}" velocity="31.67" />
-        <dynamics damping="0.1" friction="0.1" />
+        <limit effort="${max_torque}" lower="0" upper="${pi - 0.1}" velocity="31.67" />
+        <dynamics damping="0.01" friction="0.01" />
     </joint>
     <link name="knee_link">

File: ros2_ws/src/robot_description/description/torque_control.xacro (robot description, xacro)
@@ -9,7 +9,7 @@
             <inital_velocity>0</inital_velocity>
             <sub_topic>joint/hip_joint/0/cmd_torque</sub_topic>
-            <p_gain>150.0</p_gain>
-            <i_gain>0.0</i_gain>
-            <d_gain>15.0</d_gain>
+            <p_gain>100.0</p_gain>
+            <i_gain>0.01</i_gain>
+            <d_gain>25.0</d_gain>
             <i_max>1</i_max>
             <i_min>-1</i_min>
@@ -26,6 +26,6 @@
             <sub_topic>joint/knee_joint/0/cmd_torque</sub_topic>
             <p_gain>100.0</p_gain>
-            <i_gain>0.0</i_gain>
-            <d_gain>10.0</d_gain>
+            <i_gain>0.01</i_gain>
+            <d_gain>25.0</d_gain>
             <i_max>1</i_max>
             <i_min>-1</i_min>

Commit message: wrote active compliance, but something is wrong

File: ros2_ws/src/robot_description/description/robot.urdf.xacro (robot description, xacro)
@@ -41,5 +41,5 @@
         <axis xyz="0 0 1" />
         <limit effort="${max_torque}" lower="-2.8" upper="0.46" velocity="31.67" />
-        <dynamics damping="0.1" friction="0.1" />
+        <dynamics damping="0.01" friction="0.01" />
     </joint>
     <link name="hip_link">
@@ -75,5 +75,5 @@
         <axis xyz="0 0 1" />
         <limit effort="${max_torque}" lower="-2.34" upper="2.62" velocity="31.67" />
-        <dynamics damping="0.1" friction="0.1" />
+        <dynamics damping="0.01" friction="0.01" />
     </joint>
     <link name="knee_link">
