Commit message: use different controller in gz, stable gains

File: ros2_ws/src/robot_description/description/robot.urdf.xacro (robot description, xacro)
@@ -64,5 +64,5 @@
         <origin xyz="${L1_length} 0 0" rpy="0 0 0" />
         <axis xyz="0 0 1" />
-        <limit effort="${max_torque}" lower="0" upper="${pi - 0.1}" velocity="31.67" />
+        <limit effort="${max_torque}" lower="0.1" upper="${pi - 0.1}" velocity="31.67" />
         <dynamics damping="0.01" friction="0.01" />
     </joint>

File: ros2_ws/src/robot_description/description/torque_control.xacro (robot description, xacro)
@@ -2,5 +2,5 @@
 <robot xmlns:xacro="http://www.ros.org/wiki/xacro">
     <gazebo>
-        <plugin
+        <!-- <plugin
             filename="gz-sim-joint-controller-system"
             name="gz::sim::systems::JointController">
@@ -33,4 +33,14 @@
             <cmd_min>${-max_torque}</cmd_min>
             <cmd_offset>0.0</cmd_offset>
+        </plugin> -->
+        <plugin
+            filename="gz-sim-apply-joint-force-system"
+            name="gz::sim::systems::ApplyJointForce">
+            <joint_name>hip_joint</joint_name>
+        </plugin>
+        <plugin
+            filename="gz-sim-apply-joint-force-system"
+            name="gz::sim::systems::ApplyJointForce">
+            <joint_name>knee_joint</joint_name>
         </plugin>
     </gazebo>

Commit message: make urdf accurate to cad, workspace plotting

File: ros2_ws/src/robot_description/description/robot.urdf.xacro (robot description, xacro)
@@ -4,9 +4,9 @@
     <xacro:arg name="torque_control" default="false" />
     <xacro:arg name="position_control" default="false" />
-    <xacro:property name="L1_length" default="0.3"/>
+    <xacro:property name="L1_length" default="0.145" />
     <!-- <xacro:property name="L1_length" default="0.093732"/> -->
-    <xacro:property name="L2_length" default="0.25"/>
+    <xacro:property name="L2_length" default="0.215" />
     <!-- <xacro:property name="L2_length" default="0.125"/> -->
-    <xacro:property name="max_torque" default="20.1"/>
+    <xacro:property name="max_torque" default="20.1" />
     <link name="world">
     </link>
@@ -20,8 +20,17 @@
     </joint>
     <link name="base_link">
+        <visual>
+            <geometry>
+                <!-- <mesh filename="file://$(find robot_description)/meshes/base_link.stl"/> -->
+                <!-- for preview -->
+                <mesh filename="../meshes/base_link.STL" />
+                <!-- <box size="${L1_length} 0.05 0.02" /> -->
+            </geometry>
+        </visual>
         <inertial>
-            <origin xyz="0 0 0" rpy="0 0 0" />
-            <mass value="0.01" />
-            <inertia ixx="0.01" ixy="0" ixz="0" iyy="0.01" iyz="0" izz="0.01" />
+            <origin xyz="0.000113 0.003536 0.005902" rpy="0 0 0" />
+            <mass value="0.39" />
+            <inertia ixx="0.000359" ixy="0.000001" ixz="-0.000001"
+                iyy="0.000160" iyz="0.000076" izz="0.000302" />
         </inertial>
     </link>
@@ -31,15 +40,15 @@
         <origin xyz="0 0 0" rpy="${pi/2} ${pi/2} 0" />
         <axis xyz="0 0 1" />
-        <limit effort="${max_torque}" lower="-${pi}" upper="${pi}" velocity="31.67" />
+        <limit effort="${max_torque}" lower="-2.8" upper="0.46" velocity="31.67" />
         <dynamics damping="0.1" friction="0.1" />
     </joint>
     <link name="hip_link">
         <visual>
-            <origin xyz="${L1_length/2} 0 0" rpy="0 0 0" />
+            <!-- <origin xyz="${L1_length/2} 0 0" rpy="0 0 0" /> -->
             <geometry>
                 <!-- <mesh filename="file://$(find robot_description)/meshes/hip.stl"/> -->
                 <!-- for preview -->
-                <!-- <mesh filename="../meshes/hip.stl"/> -->
-                <box size="${L1_length} 0.05 0.02" />
+                <mesh filename="../meshes/hip.STL" />
+                <!-- <box size="${L1_length} 0.05 0.02" /> -->
             </geometry>
             <material name="blue">
@@ -47,14 +56,15 @@
             </material>
         </visual>
-        <collision>
-            <origin xyz="${L1_length/2} 0 0" rpy="0 0 0" />
-            <geometry>
-                <box size="${L1_length} 0.05 0.02" />
-            </geometry>
-        </collision>
+        <!-- <collision>
+            <origin xyz="${L1_length/2} 0 0" rpy="0 0 0" /> -->
+        <!-- <geometry>
+                <box size="${L1_length} 0.05 0.02" /> -->
+        <!-- </geometry> -->
+        <!-- </collision> -->
         <inertial>
-            <origin xyz="0 0 0" rpy="0 0 0" />
-            <mass value="0.6" />
-            <inertia ixx="0.01" ixy="0" ixz="0" iyy="0.01" iyz="0" izz="0.01" />
+            <origin xyz="0.016172 0.057426 0.010825" rpy="0 0 0" />
+            <mass value="0.5" />
+            <inertia ixx="0.000596" ixy=" 0.000338" ixz="-0.000138"
+                iyy="0.000959" iyz="0.000145" izz="0.001275" />
         </inertial>
     </link>
@@ -62,17 +72,17 @@
         <parent link="hip_link" />
         <child link="knee_link" />
-        <origin xyz="${L1_length} 0 0" rpy="0 0 0" />
+        <origin xyz="${L1_length} 0 0.0277" rpy="0 0 0" />
         <axis xyz="0 0 1" />
-        <limit effort="${max_torque}" lower="-${pi}" upper="${pi}" velocity="31.67" />
+        <limit effort="${max_torque}" lower="-2.34" upper="2.62" velocity="31.67" />
         <dynamics damping="0.1" friction="0.1" />
     </joint>
     <link name="knee_link">
         <visual>
-            <origin xyz="${L2_length/2} 0 0" rpy="0 0 0" />
+            <!-- <origin xyz="${L2_length/2} 0 0" rpy="0 0 0" /> -->
             <geometry>
-                <!-- <mesh filename="file://$(find robot_description)/meshes/tibia.stl"/> -->
+                <!-- <mesh filename="file://$(find robot_description)/meshes/knee.STL"/> -->
                 <!-- for preview -->
-                <!-- <mesh filename="../meshes/tibia.stl"/> -->
-                <box size="${L2_length} 0.05 0.02" />
+                <mesh filename="../meshes/knee.STL" />
+                <!-- <box size="${L2_length} 0.05 0.02" /> -->
             </geometry>
             <material name="green">
@@ -80,14 +90,15 @@
             </material>
         </visual>
-        <collision>
-            <origin xyz="${L2_length/2} 0 0" rpy="0 0 0" />
-            <geometry>
-                <box size="${L2_length} 0.01 0.04" />
-            </geometry>
-        </collision>
+        <!-- <collision> -->
+        <!-- <origin xyz="${L2_length/2} 0 0" rpy="0 0 0" /> -->
+        <!-- <geometry> -->
+        <!-- <box size="${L2_length} 0.01 0.04" /> -->
+        <!-- </geometry> -->
+        <!-- </collision> -->
         <inertial>
-            <origin xyz="0 0 0" rpy="0 0 0" />
-            <mass value="0.1" />
-            <inertia ixx="0.01" ixy="0" ixz="0" iyy="0.01" iyz="0" izz="0.01" />
+            <origin xyz="0.119035 -0.021572 0.000043" rpy="0 0 0" />
+            <mass value="0.055566" />
+            <inertia ixx="0.000022" ixy="-0.000033" ixz="0.000000"
+                iyy="0.000387" iyz="0.000000" izz="0.000407" />
         </inertial>
     </link>
@@ -95,5 +106,5 @@
     <!-- Can also change this manually in the sdf to a fixed joint -->
     <joint name="contact_joint" type="fixed">
-    <!-- <joint name="contact_joint" type="revolute"> -->
+        <!-- <joint name="contact_joint" type="revolute"> -->
         <parent link="knee_link" />
         <child link="foot_link" />
@@ -106,5 +117,8 @@
         <visual>
             <geometry>
-                <sphere radius="0.05" />
+                <!-- <mesh filename="file://$(find robot_description)/meshes/foot.stl"/> -->
+                <!-- for preview -->
+                <mesh filename="../meshes/foot.STL" />
+                <!-- <sphere radius="0.05" /> -->
             </geometry>
         </visual>
@@ -114,10 +128,12 @@
         <collision>
             <geometry>
-                <sphere radius="0.05" />
+                <cylinder radius="0.02414" length="0.01" />
             </geometry>
         </collision>
         <inertial>
-            <mass value="0.01" />
-            <inertia ixx="0.01" ixy="0" ixz="0" iyy="0.01" iyz="0" izz="0.01" />
+            <origin xyz="0.000290 -0.000906 -0.000052" rpy="0 0 0" />
+            <mass value="0.013619" />
+            <inertia ixx="0.000002" ixy="0.000000" ixz="0.000000"
+                iyy="0.000003" iyz="0.000000" izz="0.000004" />
         </inertial>
     </link>

Commit message: tune gains for new model, active compliance still buggy

File: ros2_ws/src/robot_description/description/robot.urdf.xacro (robot description, xacro)
@@ -5,10 +5,16 @@
     <xacro:arg name="position_control" default="false" />
     <xacro:property name="L1_length" default="0.145" />
-    <!-- <xacro:property name="L1_length" default="0.093732"/> -->
     <xacro:property name="L2_length" default="0.215" />
-    <!-- <xacro:property name="L2_length" default="0.125"/> -->
     <xacro:property name="max_torque" default="20.1" />
     <link name="world">
     </link>
+    <!--
+    ** IMPORTANT **
+    Moment of inertia cross terms are zero for stability
+    Moment of inertia of base_link not real because it doesn't rotate (helps sim stability)
+    Moment of inertia xx and yy terms for hip, knee, and foot are set to 0.1 for stability
+    Moment of inertia zz terms for hip, knee, and foot are multiplied by 10 for stability (if pulling
+    values from URDF, divide by 10 to get real value)
+    -->
     <joint name="slider_joint" type="prismatic">
         <parent link="world" />
@@ -22,15 +28,18 @@
         <visual>
             <geometry>
-                <!-- <mesh filename="file://$(find robot_description)/meshes/base_link.stl"/> -->
+                <mesh filename="file://$(find robot_description)/meshes/base_link.STL" />
                 <!-- for preview -->
-                <mesh filename="../meshes/base_link.STL" />
+                <!-- <mesh filename="../meshes/base_link.STL" /> -->
                 <!-- <box size="${L1_length} 0.05 0.02" /> -->
             </geometry>
+            <material name="red">
+                <color rgba="1 0 0 1" />
+            </material>
         </visual>
         <inertial>
-            <origin xyz="0.000113 0.003536 0.005902" rpy="0 0 0" />
+            <origin xyz="0.0 0 0" rpy="0 0 0" />
             <mass value="0.39" />
-            <inertia ixx="0.000359" ixy="0.000001" ixz="-0.000001"
-                iyy="0.000160" iyz="0.000076" izz="0.000302" />
+            <inertia ixx="0.1" ixy="0.0" ixz="0.0"
+                iyy="0.1" iyz="0.0" izz="0.1" />
         </inertial>
     </link>
@@ -41,5 +50,5 @@
         <axis xyz="0 0 1" />
         <limit effort="${max_torque}" lower="-2.8" upper="0.46" velocity="31.67" />
-        <dynamics damping="0.01" friction="0.01" />
+        <dynamics damping="0.1" friction="0.1" />
     </joint>
     <link name="hip_link">
@@ -47,7 +56,7 @@
             <!-- <origin xyz="${L1_length/2} 0 0" rpy="0 0 0" /> -->
             <geometry>
-                <!-- <mesh filename="file://$(find robot_description)/meshes/hip.stl"/> -->
+                <mesh filename="file://$(find robot_description)/meshes/hip.STL" />
                 <!-- for preview -->
-                <mesh filename="../meshes/hip.STL" />
+                <!-- <mesh filename="../meshes/hip.STL" /> -->
                 <!-- <box size="${L1_length} 0.05 0.02" /> -->
             </geometry>
@@ -56,15 +65,16 @@
             </material>
         </visual>
-        <!-- <collision>
-            <origin xyz="${L1_length/2} 0 0" rpy="0 0 0" /> -->
-        <!-- <geometry>
-                <box size="${L1_length} 0.05 0.02" /> -->
-        <!-- </geometry> -->
-        <!-- </collision> -->
+        <collision>
+            <geometry>
+                <mesh filename="file://$(find robot_description)/meshes/hip_collision.STL" />
+                <!-- for preview -->
+                <!-- <mesh filename="../meshes/hip_collision.STL" /> -->
+            </geometry>
+        </collision>
         <inertial>
             <origin xyz="0.016172 0.057426 0.010825" rpy="0 0 0" />
             <mass value="0.5" />
-            <inertia ixx="0.000596" ixy=" 0.000338" ixz="-0.000138"
-                iyy="0.000959" iyz="0.000145" izz="0.001275" />
+            <inertia ixx="0.01" ixy=" 0.0" ixz="0.0"
+                iyy="0.01" iyz="0.0" izz="0.01275" />
         </inertial>
     </link>
@@ -75,5 +85,5 @@
         <axis xyz="0 0 1" />
         <limit effort="${max_torque}" lower="-2.34" upper="2.62" velocity="31.67" />
-        <dynamics damping="0.01" friction="0.01" />
+        <dynamics damping="0.1" friction="0.1" />
     </joint>
     <link name="knee_link">
@@ -81,7 +91,7 @@
             <!-- <origin xyz="${L2_length/2} 0 0" rpy="0 0 0" /> -->
             <geometry>
-                <!-- <mesh filename="file://$(find robot_description)/meshes/knee.STL"/> -->
+                <mesh filename="file://$(find robot_description)/meshes/knee.STL" />
                 <!-- for preview -->
-                <mesh filename="../meshes/knee.STL" />
+                <!-- <mesh filename="../meshes/knee.STL" /> -->
                 <!-- <box size="${L2_length} 0.05 0.02" /> -->
             </geometry>
@@ -90,15 +100,16 @@
             </material>
         </visual>
-        <!-- <collision> -->
-        <!-- <origin xyz="${L2_length/2} 0 0" rpy="0 0 0" /> -->
-        <!-- <geometry> -->
-        <!-- <box size="${L2_length} 0.01 0.04" /> -->
-        <!-- </geometry> -->
-        <!-- </collision> -->
+        <collision>
+            <geometry>
+                <mesh filename="file://$(find robot_description)/meshes/knee_collision.STL" />
+                <!-- for preview -->
+                <!-- <mesh filename="../meshes/knee_collision.STL" /> -->
+            </geometry>
+        </collision>
         <inertial>
             <origin xyz="0.119035 -0.021572 0.000043" rpy="0 0 0" />
             <mass value="0.055566" />
-            <inertia ixx="0.000022" ixy="-0.000033" ixz="0.000000"
-                iyy="0.000387" iyz="0.000000" izz="0.000407" />
+            <inertia ixx="0.01" ixy="0.0" ixz="0.0"
+                iyy="0.01" iyz="0.0" izz="0.00407" />
         </inertial>
     </link>
@@ -117,9 +128,12 @@
         <visual>
             <geometry>
-                <!-- <mesh filename="file://$(find robot_description)/meshes/foot.stl"/> -->
+                <mesh filename="file://$(find robot_description)/meshes/foot.STL" />
                 <!-- for preview -->
-                <mesh filename="../meshes/foot.STL" />
+                <!-- <mesh filename="../meshes/foot.STL" /> -->
                 <!-- <sphere radius="0.05" /> -->
             </geometry>
+            <material name="red">
+                <color rgba="1 0 0 1" />
+            </material>
         </visual>
         <!-- Something is wrong with the urdf/xacro/sdf conversion.
@@ -128,5 +142,5 @@
         <collision>
             <geometry>
-                <cylinder radius="0.02414" length="0.01" />
+                <sphere radius="0.02414" />
             </geometry>
         </collision>
@@ -134,6 +148,6 @@
             <origin xyz="0.000290 -0.000906 -0.000052" rpy="0 0 0" />
             <mass value="0.013619" />
-            <inertia ixx="0.000002" ixy="0.000000" ixz="0.000000"
-                iyy="0.000003" iyz="0.000000" izz="0.000004" />
+            <inertia ixx="0.01" ixy="0.0" ixz="0.0"
+                iyy="0.01" iyz="0.0" izz="0.000004" />
         </inertial>
     </link>

File: ros2_ws/src/robot_description/description/simulation.xacro (robot description, xacro)
@@ -100,4 +100,5 @@
       name="gz::sim::systems::JointStatePublisher">
       <topic>model/robot/joint_states</topic>
+      <joint_name>slider_joint</joint_name>
       <joint_name>hip_joint</joint_name>
       <joint_name>knee_joint</joint_name>

Commit message: fix active compliance

File: ros2_ws/src/robot_description/description/robot.urdf.xacro (robot description, xacro)
@@ -28,8 +28,12 @@
         <visual>
             <geometry>
-                <mesh filename="file://$(find robot_description)/meshes/base_link.STL" />
-                <!-- for preview -->
-                <!-- <mesh filename="../meshes/base_link.STL" /> -->
-                <!-- <box size="${L1_length} 0.05 0.02" /> -->
+                <xacro:if value="$(arg use_sim_time)">
+                    <mesh filename="file://$(find robot_description)/meshes/base_link.STL" />
+                </xacro:if>
+                <xacro:unless value="$(arg use_sim_time)">
+                    <!-- for preview -->
+                    <mesh filename="../meshes/base_link.STL" />
+                    <!-- <box size="${L1_length} 0.05 0.02" /> -->
+                </xacro:unless>
             </geometry>
             <material name="red">
@@ -56,8 +60,12 @@
             <!-- <origin xyz="${L1_length/2} 0 0" rpy="0 0 0" /> -->
             <geometry>
-                <mesh filename="file://$(find robot_description)/meshes/hip.STL" />
-                <!-- for preview -->
-                <!-- <mesh filename="../meshes/hip.STL" /> -->
-                <!-- <box size="${L1_length} 0.05 0.02" /> -->
+                <xacro:if value="$(arg use_sim_time)">
+                    <mesh filename="file://$(find robot_description)/meshes/hip.STL" />
+                </xacro:if>
+                <xacro:unless value="$(arg use_sim_time)">
+                    <!-- for preview -->
+                    <mesh filename="../meshes/hip.STL" />
+                    <!-- <box size="${L1_length} 0.05 0.02" /> -->
+                </xacro:unless>
             </geometry>
             <material name="blue">
@@ -91,8 +99,12 @@
             <!-- <origin xyz="${L2_length/2} 0 0" rpy="0 0 0" /> -->
             <geometry>
-                <mesh filename="file://$(find robot_description)/meshes/knee.STL" />
-                <!-- for preview -->
-                <!-- <mesh filename="../meshes/knee.STL" /> -->
-                <!-- <box size="${L2_length} 0.05 0.02" /> -->
+                <xacro:if value="$(arg use_sim_time)">
+                    <mesh filename="file://$(find robot_description)/meshes/knee.STL" />
+                </xacro:if>
+                <xacro:unless value="$(arg use_sim_time)">
+                    <!-- for preview -->
+                    <mesh filename="../meshes/knee.STL" />
+                    <!-- <box size="${L2_length} 0.05 0.02" /> -->
+                </xacro:unless>
             </geometry>
             <material name="green">
@@ -128,8 +140,12 @@
         <visual>
             <geometry>
-                <mesh filename="file://$(find robot_description)/meshes/foot.STL" />
-                <!-- for preview -->
-                <!-- <mesh filename="../meshes/foot.STL" /> -->
-                <!-- <sphere radius="0.05" /> -->
+                <xacro:if value="$(arg use_sim_time)">
+                    <mesh filename="file://$(find robot_description)/meshes/foot.STL" />
+                </xacro:if>
+                <xacro:unless value="$(arg use_sim_time)">
+                    <!-- for preview -->
+                    <mesh filename="../meshes/foot.STL" />
+                    <!-- <sphere radius="0.05" /> -->
+                </xacro:unless>
             </geometry>
             <material name="red">

Commit message: impedence control works with base frame on top, jumping control implemented

File: ros2_ws/src/robot_description/description/robot.urdf.xacro (robot description, xacro)
@@ -22,5 +22,5 @@
         <origin xyz="0 0 1.0" rpy="0 0 0" />
         <axis xyz="0 0 1" />
-        <limit effort="0" lower="-10" upper="10" velocity="100.0" />
+        <limit effort="0" lower="-10.0" upper="10" velocity="100.0" />
         <dynamics damping="0.0" friction="0.0" />
     </joint>

Commit message: tested on hardware, leg doesn't move in straight line

File: ros2_ws/src/robot_description/description/robot.urdf.xacro (robot description, xacro)
@@ -4,5 +4,5 @@
     <xacro:arg name="torque_control" default="false" />
     <xacro:arg name="position_control" default="false" />
-    <xacro:property name="L1_length" default="0.145" />
+    <xacro:property name="L1_length" default="0.125" />
     <xacro:property name="L2_length" default="0.215" />
     <xacro:property name="max_torque" default="20.1" />
@@ -92,5 +92,5 @@
         <origin xyz="${L1_length} 0 0.0277" rpy="0 0 0" />
         <axis xyz="0 0 1" />
-        <limit effort="${max_torque}" lower="-2.34" upper="2.62" velocity="31.67" />
+        <limit effort="${max_torque}" lower="0.3" upper="2.62" velocity="31.67" />
         <dynamics damping="0.01" friction="0.01" />
     </joint>

Commit message: update urdf mass values, inertia no longer 10x

File: ros2_ws/src/robot_description/description/robot.urdf.xacro (robot description, xacro)
@@ -14,6 +14,4 @@
     Moment of inertia of base_link not real because it doesn't rotate (helps sim stability)
     Moment of inertia xx and yy terms for hip, knee, and foot are set to 0.1 for stability
-    Moment of inertia zz terms for hip, knee, and foot are multiplied by 10 for stability (if pulling
-    values from URDF, divide by 10 to get real value)
     -->
     <joint name="slider_joint" type="prismatic">
@@ -43,5 +41,5 @@
         <inertial>
             <origin xyz="0.0 0 0" rpy="0 0 0" />
-            <mass value="0.39" />
+            <mass value="0.67115" />
             <inertia ixx="0.1" ixy="0.0" ixz="0.0"
                 iyy="0.1" iyz="0.0" izz="0.1" />
@@ -81,8 +79,8 @@
         </collision>
         <inertial>
-            <origin xyz="0.016172 0.057426 0.010825" rpy="0 0 0" />
-            <mass value="0.5" />
+            <origin xyz="0.014130 0.059212 0.010598" rpy="0 0 0" />
+            <mass value="0.482069" />
             <inertia ixx="0.01" ixy=" 0.0" ixz="0.0"
-                iyy="0.01" iyz="0.0" izz="0.01275" />
+                iyy="0.01" iyz="0.0" izz="0.001186" />
         </inertial>
     </link>
@@ -120,8 +118,8 @@
         </collision>
         <inertial>
-            <origin xyz="0.119035 -0.021572 0.000043" rpy="0 0 0" />
-            <mass value="0.055566" />
+            <origin xyz="0.117055 -0.019215 -0.000018" rpy="0 0 0" />
+            <mass value="0.047151" />
             <inertia ixx="0.01" ixy="0.0" ixz="0.0"
-                iyy="0.01" iyz="0.0" izz="0.00407" />
+                iyy="0.01" iyz="0.0" izz="0.000464" />
         </inertial>
     </link>
