Commit message: cant name package robot_description or else ros2_control has trouble finding config file

File: ros2_ws/src/robot_desc/description/robot.urdf.xacro (robot description, xacro)
@@ -38,5 +38,5 @@
             <origin xyz="${L1_length/2} 0 0" rpy="0 0 0" />
             <geometry>
-                <!-- <mesh filename="file://$(find robot_description)/meshes/hip.stl"/> -->
+                <!-- <mesh filename="file://$(find robot_desc)/meshes/hip.stl"/> -->
                 <!-- for preview -->
                 <!-- <mesh filename="../meshes/hip.stl"/> -->
@@ -71,5 +71,5 @@
             <origin xyz="${L2_length/2} 0 0" rpy="0 0 0" />
             <geometry>
-                <!-- <mesh filename="file://$(find robot_description)/meshes/tibia.stl"/> -->
+                <!-- <mesh filename="file://$(find robot_desc)/meshes/tibia.stl"/> -->
                 <!-- for preview -->
                 <!-- <mesh filename="../meshes/tibia.stl"/> -->
@@ -123,12 +123,12 @@
     </link>
     <xacro:if value="$(arg use_sim_time)">
-        <xacro:include filename="$(find robot_description)/description/simulation.xacro" />
+        <xacro:include filename="$(find robot_desc)/description/simulation.xacro" />
         <xacro:if value="$(arg torque_control)">
-            <xacro:include filename="$(find robot_description)/description/torque_control.xacro" />
+            <xacro:include filename="$(find robot_desc)/description/torque_control.xacro" />
         </xacro:if>
         <!-- <xacro:if value="$(arg position_control)"> -->
-            <!-- <xacro:include filename="$(find robot_description)/description/position_control.xacro" /> -->
+            <!-- <xacro:include filename="$(find robot_desc)/description/position_control.xacro" /> -->
         <!-- </xacro:if> -->
-        <!-- <xacro:include filename="$(find robot_description)/description/ros2_control.xacro" /> -->
+        <xacro:include filename="$(find robot_desc)/description/ros2_control.xacro" />
     </xacro:if>
 </robot>

File: ros2_ws/src/robot_desc/description/ros2_control.xacro (robot description, xacro)
@@ -26,5 +26,5 @@
             filename="libgz_ros2_control-system.so"
             name="gz_ros2_control::GazeboSimROS2ControlPlugin">
-            <parameters>$(find robot_description)/config/ros2_control.yaml</parameters>
+            <parameters>$(find robot_desc)/config/ros2_control.yaml</parameters>
         </plugin>
     </gazebo>
